File: kicad/IntelligentTrafficLight.kicad_pcb (KiCad board)
At the start: 4 copper layers, 100 x 140 mm, 136 parts, among them J1 USB-C Receptacle, J2 Conn_01x07_Socket, J3 Conn_01x10_Socket, J4 Conn_01x07_Socket, J5 Conn_01x03_Pin, Q2 AO3415, SW1 Pushbutton, SW3 Pushbutton, U1 ESP32-C3-MINI-1-H4X, U2 TLV76133DCY, U3 PCA9685PW, U4 TLC555xD, U5 TLC555xD, U6 TLC555xD

Commit message: add comments to kicad schematic
Parts:
- removed C31, C34: 100nF, Capacitor_SMD:C_0402_1005Metric
- removed C32: 10uF, Capacitor_SMD:C_0402_1005Metric
- removed C33: 1uF, Capacitor_SMD:C_0402_1005Metric
- removed GND (x2): TestPoint, Connector_PinSocket_2.54mm:PinSocket_1x01_P2.54mm_Vertical
- removed JP10, JP11: SolderJumper_2_Bridged, Jumper:SolderJumper-2_P1.3mm_Bridged_RoundedPad1.0x1.5mm
- removed Q2: AO3415, Package_TO_SOT_SMD:SOT-23
- removed R39: 10k, Resistor_SMD:R_0402_1005Metric
- removed R40, R41: 0, Resistor_SMD:R_0402_1005Metric
- removed REF** (x3): Smolhaj_Scale_0.1, Symbol:Smolhaj_Scale_0.1
- removed SW3: Pushbutton, EASYEDA2KICAD:SW-SMD_6P-L5.2-W5.2-P3.70-LS6.4
- added JP3: SolderJumper_2_Open, Jumper:SolderJumper-2_P1.3mm_Open_RoundedPad1.0x1.5mm, F.Cu at (188.5, 120.2)
- added JP4: SolderJumper_2_Bridged, Jumper:SolderJumper-2_P1.3mm_Bridged_RoundedPad1.0x1.5mm, F.Cu at (178.0, 120.3)
- added SW2: Pushbutton, EASYEDA2KICAD:SW-SMD_6P-L5.2-W5.2-P3.70-LS6.4, F.Cu at (190.3, 115.2)
- added U7: TLC555xD, Package_SO:SOIC-8_3.9x4.9mm_P1.27mm, F.Cu at (180.1, 115.3)
- C1: value 1nF -> 10uF; footprint Capacitor_THT:C_Radial_D5.0mm_H11.0mm_P2.00mm -> Capacitor_SMD:C_0402_1005Metric
- C10: value 10uF -> 22uF; footprint Capacitor_SMD:C_0402_1005Metric -> Capacitor_SMD:C_0805_2012Metric
- C11, C9: value 100nF -> 22uF; footprint Capacitor_SMD:C_0402_1005Metric -> Capacitor_SMD:C_0805_2012Metric
- C12, C20: value 250nF -> 100nF
- C13, C14: value C -> 1nF
- C15: value 1nF -> 10nF; footprint Capacitor_THT:C_Radial_D5.0mm_H11.0mm_P2.00mm -> Capacitor_SMD:C_0402_1005Metric
- C18: value 10uF -> 1nF
- C19: value 100nF -> 10uF
- C2: value 10nF -> 100nF
- C21, C28: value C -> 10uF; footprint Capacitor_THT:C_Radial_D5.0mm_H11.0mm_P2.00mm -> Capacitor_SMD:C_0402_1005Metric
- C22: value 1nF -> 100nF; footprint Capacitor_THT:C_Radial_D5.0mm_H11.0mm_P2.00mm -> Capacitor_SMD:C_0402_1005Metric
- C23: value 10nF -> 250nF; footprint Capacitor_SMD:C_0402_1005Metric -> Capacitor_THT:C_Radial_D5.0mm_H11.0mm_P2.00mm
- C24: value 1nF -> 250nF; footprint Capacitor_SMD:C_0402_1005Metric -> Capacitor_THT:C_Radial_D5.0mm_H11.0mm_P2.00mm
- C25: value 10uF -> 1nF; footprint Capacitor_SMD:C_0402_1005Metric -> Capacitor_THT:C_Radial_D5.0mm_H11.0mm_P2.00mm
- C26: value 100nF -> 10nF
- C27: value 250nF -> 1nF
- C29: value C -> 100nF; footprint Capacitor_THT:C_Radial_D5.0mm_H11.0mm_P2.00mm -> Capacitor_SMD:C_0402_1005Metric
- C3: value 1nF -> 1uF
- C30: value C -> 250nF
- C5: value 10uF -> 100nF
- C8: value 22uF -> 10uF; footprint Capacitor_SMD:C_0603_1608Metric -> Capacitor_SMD:C_0402_1005Metric
- D2: value TPD3E001DRYR -> LED; footprint Package_SON:Texas_USON-6_1x1.45mm_P0.5mm_SMD -> LED_THT:LED_D5.0mm
- D4: value LED -> TPD3E001DRYR; footprint LED_THT:LED_D5.0mm -> Package_SON:Texas_USON-6_1x1.45mm_P0.5mm_SMD
- J1: value USB-C Receptacle -> Conn_01x03_Pin; footprint Connector_USB:USB_C_Receptacle_G-Switch_GT-USB-7010ASV -> Connector_PinHeader_1.00mm:PinHeader_1x03_P1.00mm_Vertical
- J2: value Conn_01x07_Socket -> Conn_01x10_Socket; footprint Connector_PinSocket_2.54mm:PinSocket_1x07_P2.54mm_Horizontal -> Connector_PinSocket_2.54mm:PinSocket_1x10_P2.54mm_Horizontal
- J3: value Conn_01x10_Socket -> USB-C Receptacle; footprint Connector_PinSocket_2.54mm:PinSocket_1x10_P2.54mm_Horizontal -> Connector_USB:USB_C_Receptacle_G-Switch_GT-USB-7010ASV
- J5: value Conn_01x03_Pin -> Conn_01x07_Socket; footprint Connector_PinHeader_1.00mm:PinHeader_1x03_P1.00mm_Vertical -> Connector_PinSocket_2.54mm:PinSocket_1x07_P2.54mm_Horizontal
- JP1, JP2: value SolderJumper_2_Bridged -> SolderJumper_2_Open; footprint Jumper:SolderJumper-2_P1.3mm_Bridged_RoundedPad1.0x1.5mm -> Jumper:SolderJumper-2_P1.3mm_Open_RoundedPad1.0x1.5mm
- JP7, JP8, JP9: value SolderJumper_2_Open -> SolderJumper_2_Bridged; footprint Jumper:SolderJumper-2_P1.3mm_Open_RoundedPad1.0x1.5mm -> Jumper:SolderJumper-2_P1.3mm_Bridged_RoundedPad1.0x1.5mm
- R1: value 510 -> 10k
- R10, R15: value 510 -> 50
- R11, R16: value 200 -> 50
- R12, R17: value 200 -> 50; footprint Resistor_THT:R_Axial_DIN0207_L6.3mm_D2.5mm_P10.16mm_Horizontal -> Resistor_SMD:R_0402_1005Metric
- R13, R18: value 3.3k -> 50
- R14, R19: value 6.8k -> 50
- R2: value 200 -> 10k
- R25, R26: value 50 -> 5.1k 1%
- R27, R28: value 50 -> 0
- R29: value 50 -> 5k
- R3: value 200 -> 10k; footprint Resistor_THT:R_Axial_DIN0207_L6.3mm_D2.5mm_P10.16mm_Horizontal -> Resistor_SMD:R_0402_1005Metric
- R30: value 50 -> 5k; footprint Resistor_SMD:R_0402_1005Metric -> Resistor_THT:R_Axial_DIN0207_L6.3mm_D2.5mm_P10.16mm_Horizontal
- R31, R33: value 50 -> 1k
- R32, R34: value 50 -> 1.5k
- R35: value 10k -> 0
- R36: value 22 -> 5k
- R37: value 22 -> 1k
- R38: value 10k -> 1.5k
- R4: value 3.3k -> 22
- R5: value 6.8k -> 10k
- R6: value 10k -> 22
- R7, R8: value 5.1k 1% -> 0
- U2: value TLV76133DCY -> PCA9685PW; footprint Package_TO_SOT_SMD:SOT-223-3_TabPin2 -> Package_SO:TSSOP-28_4.4x9.7mm_P0.65mm
- U3: value PCA9685PW -> TLV76133DCY; footprint Package_SO:TSSOP-28_4.4x9.7mm_P0.65mm -> Package_TO_SOT_SMD:SOT-223-3_TabPin2
- U4: value TLC555xD -> MAX40200AUK; footprint Package_SO:SOIC-8_3.9x4.9mm_P1.27mm -> Package_TO_SOT_SMD:SOT-23-5
Connections:
- AE1 pad 1: Net-(JP2-A) -> Net-(JP6-A)
- AE1 pad 2: Net-(JP1-A) -> Net-(JP4-A)
- AE2 pad 1: Net-(JP5-A) -> Net-(JP7-A)
- AE2 pad 2: Net-(JP6-A) -> Net-(JP5-A)
- AE3 pad 1: Net-(JP11-A) -> Net-(JP9-A)
- AE3 pad 2: Net-(JP10-A) -> Net-(JP8-A)
- C1 pad 1: Net-(JP1-B) -> +3.3V
- C10 pad 1: GND -> +3.3V
- C10 pad 2: +3.3V -> GND
- C11 pad 1: GND -> +3.3V
- C11 pad 2: +5V -> GND
- C12 pad 1: Net-(JP1-B) -> GND
- C12 pad 2: Net-(JP2-B) -> /VBUS_{fused}
- C13 pad 1: Net-(JP1-B) -> Net-(JP4-B)
- C13 pad 2: Net-(JP2-B) -> GND
- C14 pad 1: Net-(JP1-B) -> Net-(JP5-B)
- C14 pad 2: Net-(JP2-B) -> GND
- C15 pad 1: Net-(JP6-B) -> GND
- C15 pad 2: GND -> Net-(U5-CV)
- C16 pad 2: Net-(U5-CV) -> Net-(U6-CV)
- C17 pad 1: Net-(JP6-B) -> Net-(JP4-B)
- C18 pad 1: GND -> Net-(JP5-B)
- C18 pad 2: +5V -> GND
- C2 pad 1: GND -> +3.3V
- C2 pad 2: Net-(U4-CV) -> GND
- C20 pad 1: Net-(JP6-B) -> GND
- C20 pad 2: Net-(JP5-B) -> +5V
- C21 pad 1: Net-(JP6-B) -> GND
- C21 pad 2: Net-(JP5-B) -> +5V
- C22 pad 1: Net-(JP10-B) -> GND
- C22 pad 2: GND -> +5V
- C23 pad 1: GND -> Net-(JP4-B)
- C23 pad 2: Net-(U6-CV) -> Net-(JP6-B)
- C24 pad 1: Net-(JP10-B) -> Net-(JP5-B)
- C24 pad 2: GND -> Net-(JP7-B)
- C25 pad 1: GND -> Net-(JP8-B)
- C25 pad 2: +5V -> GND
- C26 pad 2: +5V -> Net-(U7-CV)
- C27 pad 1: Net-(JP10-B) -> Net-(JP8-B)
- C27 pad 2: Net-(JP11-B) -> GND
- C28 pad 1: Net-(JP6-B) -> GND
- C28 pad 2: Net-(JP5-B) -> +5V
- C29 pad 1: Net-(JP10-B) -> GND
- C29 pad 2: Net-(JP11-B) -> +5V
- C3 pad 1: Net-(JP1-B) -> GND
- C3 pad 2: GND -> /EN
- C30 pad 1: Net-(JP10-B) -> Net-(JP8-B)
- C30 pad 2: Net-(JP11-B) -> Net-(JP9-B)
- C4 pad 1: VBUS_{unregulated} -> GND
- C4 pad 2: GND -> +3.3V
- C5 pad 1: +3.3V -> GND
- C5 pad 2: GND -> +3.3V
- C6 pad 1: +3.3V -> GND
- C6 pad 2: GND -> Net-(C6-Pad2)
- C7 pad 1: GND -> VBUS_{unregulated}
- C7 pad 2: +5V -> GND
- C8 pad 1: VBUS_{unregulated} -> +3.3V
- C9 pad 1: GND -> +3.3V
- C9 pad 2: /VBUS_{fused} -> GND
- D2 pad 1: /USB D- -> Net-(D2-K)
- D2 pad 2: /USB D+ -> +3.3V
- D4 pad 1: Net-(D4-K) -> /USB D-
- D4 pad 2: +3.3V -> /USB D+
- J2 pad 1: +3.3V -> Net-(J2-Pin_1)
- J2 pad 2: GND -> Net-(J2-Pin_2)
- J2 pad 3: /LOOP_OUT_1 -> Net-(J2-Pin_3)
- J2 pad 4: /LOOP_OUT_2 -> Net-(J2-Pin_4)
- J2 pad 5: /LOOP_OUT_3 -> Net-(J2-Pin_5)
- J2 pad 6: GND -> Net-(J2-Pin_6)
- J2 pad 7: VBUS_{unregulated} -> Net-(J2-Pin_7)
- J5 pad 1: Net-(D1-K) -> +3.3V
- J5 pad 2: Net-(D3-K) -> GND
- J5 pad 3: Net-(D4-K) -> /LOOP_OUT_1
- JP1 pad 1: Net-(JP1-A) -> /GPIO_5
- JP1 pad 2: Net-(JP1-B) -> /LOOP_OUT_1
- JP2 pad 1: Net-(JP2-A) -> /GPIO_6
- JP2 pad 2: Net-(JP2-B) -> /LOOP_OUT_2
- JP7 pad 1: /GPIO_5 -> Net-(JP7-A)
- JP7 pad 2: /LOOP_OUT_1 -> Net-(JP7-B)
- JP8 pad 1: /GPIO_6 -> Net-(JP8-A)
- JP8 pad 2: /LOOP_OUT_2 -> Net-(JP8-B)
- JP9 pad 1: /GPIO_7 -> Net-(JP9-A)
- JP9 pad 2: /LOOP_OUT_3 -> Net-(JP9-B)
- R1 pad 1: +5V -> +3.3V
- R1 pad 2: Net-(U4-DIS) -> /EN
- R10 pad 1: +5V -> Net-(U2-LED1)
- R10 pad 2: Net-(U5-DIS) -> Net-(D2-K)
- R11 pad 1: Net-(U5-DIS) -> Net-(U2-LED2)
- R11 pad 2: Net-(JP5-B) -> Net-(D3-K)
- R12 pad 1: Net-(U5-DIS) -> Net-(U2-LED3)
- R12 pad 2: Net-(JP5-B) -> Net-(J2-Pin_1)
- R13 pad 1: /Inductive Loop/OUT3 -> Net-(U2-LED4)
- R13 pad 2: /LOOP_OUT_3 -> Net-(J2-Pin_2)
- R14 pad 1: /LOOP_OUT_3 -> Net-(U2-LED5)
- R14 pad 2: GND -> Net-(J2-Pin_3)
- R15 pad 1: +5V -> Net-(U2-LED6)
- R15 pad 2: Net-(U6-DIS) -> Net-(J2-Pin_4)
- R16 pad 1: Net-(U6-DIS) -> Net-(U2-LED7)
- R16 pad 2: Net-(JP11-B) -> Net-(J2-Pin_5)
- R17 pad 1: Net-(U6-DIS) -> Net-(U2-LED8)
- R17 pad 2: Net-(JP11-B) -> Net-(J2-Pin_6)
- R18 pad 1: /Inductive Loop/OUT1 -> Net-(U2-LED9)
- R18 pad 2: /LOOP_OUT_1 -> Net-(J2-Pin_7)
- R19 pad 1: /LOOP_OUT_1 -> Net-(U2-LED10)
- R19 pad 2: GND -> Net-(J2-Pin_8)
- R2 pad 1: Net-(U4-DIS) -> +3.3V
- R2 pad 2: Net-(JP2-B) -> /GPIO_8
- R20 pad 1: Net-(U3-LED1) -> Net-(U2-LED11)
- R20 pad 2: Net-(D3-K) -> Net-(J2-Pin_9)
- R21 pad 1: Net-(U3-LED2) -> Net-(U2-LED12)
- R21 pad 2: Net-(D4-K) -> Net-(J2-Pin_10)
- R22 pad 1: Net-(U3-LED3) -> Net-(U2-LED13)
- R22 pad 2: Net-(J3-Pin_1) -> unconnected-(R22-Pad2)
- R23 pad 1: Net-(U3-LED4) -> Net-(U2-LED14)
- R23 pad 2: Net-(J3-Pin_2) -> unconnected-(R23-Pad2)
- R24 pad 1: Net-(U3-LED5) -> Net-(U2-LED15)
- R24 pad 2: Net-(J3-Pin_3) -> unconnected-(R24-Pad2)
- R25 pad 1: Net-(U3-LED6) -> GND
- R25 pad 2: Net-(J3-Pin_4) -> Net-(J3-CC1)
- R26 pad 1: Net-(U3-LED7) -> GND
- R26 pad 2: Net-(J3-Pin_5) -> Net-(J3-CC2)
- R27 pad 1: Net-(U3-LED8) -> Net-(U5-DIS)
- R27 pad 2: Net-(J3-Pin_6) -> Net-(JP6-B)
- R28 pad 1: Net-(U3-LED9) -> Net-(U6-DIS)
- R28 pad 2: Net-(J3-Pin_7) -> Net-(JP7-B)
- R29 pad 1: Net-(U3-LED10) -> +5V
- R29 pad 2: Net-(J3-Pin_8) -> Net-(U5-DIS)
- R3 pad 1: Net-(U4-DIS) -> /GPIO_8
- R3 pad 2: Net-(JP2-B) -> +3.3V
- R30 pad 1: Net-(U3-LED11) -> +5V
- R30 pad 2: Net-(J3-Pin_9) -> Net-(U6-DIS)
- R31 pad 1: Net-(U3-LED12) -> /Inductive Loop/OUT2
- R31 pad 2: Net-(J3-Pin_10) -> /LOOP_OUT_2
- R32 pad 1: Net-(U3-LED13) -> /LOOP_OUT_2
- R32 pad 2: unconnected-(R32-Pad2) -> GND
- R33 pad 1: Net-(U3-LED14) -> /Inductive Loop/OUT1
- R33 pad 2: unconnected-(R33-Pad2) -> /LOOP_OUT_1
- R34 pad 1: Net-(U3-LED15) -> /LOOP_OUT_1
- R34 pad 2: unconnected-(R34-Pad2) -> GND
- R35 pad 1: +3.3V -> Net-(U7-DIS)
- R35 pad 2: /EN -> Net-(JP9-B)
- R36 pad 1: Net-(U1-IO19) -> +5V
- R36 pad 2: /USB D+ -> Net-(U7-DIS)
- R37 pad 1: /USB D- -> /Inductive Loop/OUT3
- R37 pad 2: Net-(U1-IO18) -> /LOOP_OUT_3
- R38 pad 1: +3.3V -> /LOOP_OUT_3
- R38 pad 2: Net-(U1-IO2) -> GND
- R4 pad 1: /Inductive Loop/OUT2 -> /USB D-
- R4 pad 2: /LOOP_OUT_2 -> Net-(U1-IO18)
- R5 pad 1: /LOOP_OUT_2 -> +3.3V
- R5 pad 2: GND -> Net-(U1-IO2)
- R6 pad 1: /GPIO_8 -> Net-(U1-IO19)
- R6 pad 2: +3.3V -> /USB D+
- R7 pad 1: GND -> /EN
- R7 pad 2: Net-(J1-CC1) -> Net-(C6-Pad2)
- R8 pad 1: GND -> /GPIO_0
- R8 pad 2: Net-(J1-CC2) -> Net-(R8-Pad2)
- R9 pad 1: Net-(U3-LED0) -> Net-(U2-LED0)
- RV1 pad 2: Net-(JP2-B) -> Net-(U5-DIS)
- RV1 pad 3: Net-(U4-DIS) -> +5V
- RV2 pad 2: Net-(JP5-B) -> Net-(U6-DIS)
- RV2 pad 3: Net-(U5-DIS) -> +5V
- RV3 pad 2: Net-(JP11-B) -> Net-(U7-DIS)
- RV3 pad 3: Net-(U6-DIS) -> +5V
- SW1 pad 1: Net-(R41-Pad2) -> Net-(C6-Pad2)
- TP10 pad 1: Net-(JP2-A) -> Net-(JP8-A)
- TP11 pad 1: Net-(JP1-A) -> Net-(JP8-A)
- TP12 pad 1: Net-(JP6-A) -> Net-(JP9-A)
- TP13 pad 1: Net-(JP5-A) -> Net-(JP9-A)
- TP2 pad 1: Net-(JP1-A) -> Net-(JP4-A)
- TP3 pad 1: Net-(JP2-A) -> Net-(JP5-A)
- TP4 pad 1: Net-(JP10-A) -> Net-(JP4-A)
- TP5 pad 1: Net-(JP11-A) -> Net-(JP5-A)
- TP6 pad 1: Net-(JP5-A) -> Net-(JP6-A)
- TP7 pad 1: Net-(JP10-A) -> Net-(JP7-A)
- TP9 pad 1: Net-(JP11-A) -> Net-(JP7-A)
- U2 pad 1: GND -> +3.3V
- U2 pad 2: +3.3V -> GND
- U2 pad 3: VBUS_{unregulated} -> +3.3V
- U3 pad 1: +3.3V -> GND
- U3 pad 2: GND -> +3.3V
- U3 pad 3: +3.3V -> VBUS_{unregulated}
- U4 pad 1: GND -> /VBUS_{fused}
- U4 pad 2: Net-(JP1-B) -> GND
- U4 pad 3: /Inductive Loop/OUT2 -> /VBUS_{fused}
- U4 pad 4: +5V -> unconnected-(U4-NC-Pad4)
- U4 pad 5: Net-(U4-CV) -> +5V
- U5 pad 2: Net-(JP6-B) -> Net-(JP4-B)
- U5 pad 3: /Inductive Loop/OUT3 -> /Inductive Loop/OUT2
- U5 pad 6: Net-(JP6-B) -> Net-(JP4-B)
- U6 pad 2: Net-(JP10-B) -> Net-(JP5-B)
- U6 pad 6: Net-(JP10-B) -> Net-(JP5-B)
Routing:
- net (no net): track 0.00 -> 441.3 mm, vias 0 -> 1
- net +5V: track 115.3 -> 199.1 mm, vias 6 -> 12
- net Net-(JP10-A): track 75.5 -> 0.00 mm, vias 1 -> 0
- net /USB D-: track 76.4 -> 2.68 mm, vias 3 -> 0
- net /Inductive Loop/OUT3: track 3.39 -> 76.4 mm, vias 0 -> 3
- net /GPIO_5: track 62.6 -> 135.4 mm, vias 2 -> 3
- net Net-(JP1-A): track 72.9 -> 0.00 mm, vias 1 -> 0
- net +3.3V: track 45.4 -> 117.6 mm, vias 9 -> 14
- net /USB D+: track 71.7 -> 4.47 mm, vias 4 -> 1
- net Net-(U3-LED0): track 59.6 -> 0.00 mm, vias 2 -> 0
- net Net-(U2-LED0): track 0.00 -> 59.6 mm, vias 0 -> 2
- net Net-(JP11-A): track 54.9 -> 0.00 mm
- net Net-(JP2-B): track 54.5 -> 0.00 mm
- net Net-(JP2-A): track 52.6 -> 0.00 mm
- net Net-(JP11-B): track 51.5 -> 0.00 mm, vias 1 -> 0
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
Commit message: update!
Parts:
- removed C6: 100nF, Capacitor_SMD:C_0402_1005Metric
- removed C8: 10uF, Capacitor_SMD:C_0402_1005Metric
- removed C9: 22uF, Capacitor_SMD:C_0805_2012Metric
- removed D2: LED, LED_THT:LED_D5.0mm
- removed F1: 1.5A, Fuse:Fuse_1206_3216Metric_Pad1.42x1.75mm_HandSolder
- removed J1: Conn_01x03_Pin, Connector_PinHeader_1.00mm:PinHeader_1x03_P1.00mm_Vertical
- removed R35, R7, R8: 0, Resistor_SMD:R_0402_1005Metric
- removed R36: 5k, Resistor_SMD:R_0402_1005Metric
- removed R37: 1k, Resistor_SMD:R_0402_1005Metric
- removed R38: 1.5k, Resistor_SMD:R_0402_1005Metric
- removed TP1: VBUS, Connector_PinSocket_2.54mm:PinSocket_1x01_P2.54mm_Vertical
- removed U1: ESP32-C3-MINI-1-H4X, EASYEDA2KICAD:WIFIM-SMD_ESP32-C3-MINI-1
- C1, C10, C11, C12, C13, C14, C15, C16, C17, C18, C19, C2, C20, C21, C22, C23, C24, C25, C26, C27, C28, C29, C3, C30, C4, C5, C7, D1, D3, D4, H3, H4, J2, J3, J4, JP1, JP2, JP3, JP4, JP5, JP6, JP7, JP8, JP9, R1, R10, R11, R12, R13, R14, R15, R16, R17, R18, R19, R2, R20, R21, R22, R23, R24, R25, R26, R27, R28, R29, R3, R30, R31, R32, R33, R34, R4, R5, R6, R9, RV1, RV2, RV3, SW1, SW2, TP10, TP11, TP12, TP13, TP2, TP3, TP4, TP5, TP6, TP7, TP8, TP9, U2, U3, U4, U5, U6, U7: moved to B.Cu
- J5, kibuzzard-691CE1C1: moved to F.Cu
- moved H4 202.5 mm to (270.1, 142.8), turned to 180 degrees
- moved TP4 198.0 mm to (267.8, 94.8), turned to 180 degrees
- moved TP7 198.0 mm to (267.8, 76.8)
- moved C22 194.5 mm to (266.1, 106.7)
- moved C27 193.7 mm to (265.7, 103.5), turned to 180 degrees
- moved TP5 190.6 mm to (264.1, 94.8), turned to 180 degrees
- moved JP7 187.3 mm to (262.4, 120.8), turned to 180 degrees
- moved TP9 187.1 mm to (262.3, 76.8), turned to 180 degrees
- moved C23 186.6 mm to (262.1, 107.8)
- moved C29 185.7 mm to (261.7, 117.6)
- moved R19 185.7 mm to (261.7, 96.6)
- moved R18 184.6 mm to (261.1, 99.1), turned to 0 degrees
- moved C24 180.6 mm to (259.1, 111.7)
- moved U6 179.6 mm to (258.6, 105.8)
- moved R15 176.6 mm to (257.1, 111.7), turned to 0 degrees
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Routing:
- net (no net): track 441.3 -> 0.00 mm
- net GND: track 366.9 -> 0.00 mm, vias 83 -> 81
- net +5V: track 199.1 -> 0.00 mm, vias 12 -> 10
- net /GPIO_5: track 135.4 -> 0.00 mm
- net /LOOP_OUT_1: track 126.9 -> 0.00 mm
- net +3.3V: track 117.6 -> 0.00 mm, vias 14 -> 16
- net VBUS_{unregulated}: track 94.8 -> 0.00 mm, vias 4 -> 3
- net Net-(JP6-A): track 76.6 -> 0.00 mm
- net /Inductive Loop/OUT3: track 76.4 -> 0.00 mm, vias 3 -> 4
- net /LOOP_OUT_3: track 75.7 -> 0.00 mm
- net /LOOP_OUT_2: track 70.3 -> 0.00 mm, vias 3 -> 2
- net Net-(U2-LED0): track 59.6 -> 0.00 mm
- net Net-(U5-DIS): track 57.6 -> 0.00 mm
- net Net-(JP5-B): track 56.9 -> 0.00 mm
- net Net-(JP5-A): track 56.7 -> 0.00 mm
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- added copper zone on B.Cu, net +3.3V
- added copper zone on In2.Cu, net +3.3V
- added copper zone on B.Cu, net VBUS_{unregulated}
- removed copper zone on F.Cu, net +3.3V
- removed copper zone on F.Cu, net VBUS_{unregulated}
Other:
- board size 100 x 140 mm -> 100 x 100 mm

Commit message: nothing
Parts:
- removed the C25 at (254.1, 105.8)
- removed the C30 at (255.7, 117.6)
- removed the D4 at (235.1, 126.3)
- removed the JP1 at (205.1, 96.6)
- removed the JP2 at (202.1, 96.6)
- removed the JP3 at (209.6, 145.2)
- removed the R3 at (190.2, 93.8)
- removed kibuzzard-691CE1C1: G***, kibuzzard-691CE1C1
- added C15: 10uF, Capacitor_SMD:C_0402_1005Metric, F.Cu at (373.2, 122.5)
- added C16: 22uF, Capacitor_SMD:C_0805_2012Metric, F.Cu at (369.5, 123.0)
- added C17: 22uF, Capacitor_SMD:C_0805_2012Metric, F.Cu at (369.5, 126.0)
- added C18: 22uF, Capacitor_SMD:C_0805_2012Metric, F.Cu at (369.5, 129.0)
- added C19: 10uF, Capacitor_SMD:C_0402_1005Metric, F.Cu at (373.2, 124.5)
- added C20: 100nF, Capacitor_SMD:C_0402_1005Metric, F.Cu at (373.2, 132.3)
- added C21: 100nF, Capacitor_SMD:C_0402_1005Metric, F.Cu at (373.2, 134.3)
- added C22: 1uF, Capacitor_SMD:C_0402_1005Metric, F.Cu at (202.0, 102.8)
- added C6: 100nF, Capacitor_SMD:C_0402_1005Metric, F.Cu at (137.6, 154.3)
- added C8: 8.2pF, Capacitor_SMD:C_0402_1005Metric, F.Cu at (137.6, 156.2)
- added C9: 8.2pF, Capacitor_SMD:C_0402_1005Metric, F.Cu at (137.6, 158.2)
- added D1: LED, LED_THT:LED_D5.0mm, F.Cu at (80.1, 138.1)
- added D3: LED, LED_THT:LED_D5.0mm, F.Cu at (382.5, 65.3)
- added D5: TT0314TPX, easyeda2kicad:DFN2510-10_L2.5-W1.0-P0.50-BL, F.Cu at (359.7, 100.3)
- added D6: LED, LED_THT:LED_D5.0mm, F.Cu at (382.5, 72.8)
- added D7: LED, LED_THT:LED_D5.0mm, F.Cu at (369.7, 117.8)
- added D8: TPD3E001DRYR, Package_SON:Texas_USON-6_1x1.45mm_P0.5mm_SMD, F.Cu at (203.8, 102.8)
- added F1: 750mA Hold, 1.5A trip, polyfuse, Fuse:Fuse_1812_4532Metric, F.Cu at (381.0, 124.0)
- added F2: 1.5A, Fuse:Fuse_1206_3216Metric_Pad1.42x1.75mm_HandSolder, F.Cu at (208.5, 107.3)
- added FB1: FerriteBead R600, Inductor_SMD:L_0603_1608Metric, F.Cu at (395.2, 79.8)
- added J1: JTAG ESP-Prog, Connector_PinSocket_2.54mm:PinSocket_1x10_P2.54mm_Horizontal, F.Cu at (192.4, 29.9)
- added J4: Conn_02x07_Top_Bottom, Connector_PinSocket_2.54mm:PinSocket_2x07_P2.54mm_Horizontal, F.Cu at (216.0, 50.0)
- added J5: Conn_01x03_Pin, Connector_PinHeader_1.00mm:PinHeader_1x03_P1.00mm_Vertical, F.Cu at (363.7, 89.6)
- added J8: USB-C Receptacle, Connector_USB:USB_C_Receptacle_G-Switch_GT-USB-7010ASV, F.Cu at (224.1, 103.6)
- added JP5: SolderJumper_2_Open, Jumper:SolderJumper-2_P1.3mm_Open_RoundedPad1.0x1.5mm, F.Cu at (389.0, 105.7)
- added JP6: SolderJumper_2_Open, Jumper:SolderJumper-2_P1.3mm_Open_RoundedPad1.0x1.5mm, F.Cu at (389.0, 109.3)
- added JP9: SolderJumper_2_Open, Jumper:SolderJumper-2_P1.3mm_Open_RoundedPad1.0x1.5mm, F.Cu at (389.0, 112.8)
- added Q1: S8050, Package_TO_SOT_THT:TO-92_Inline, F.Cu at (399.2, 81.8)
- added Q2: S8050, Package_TO_SOT_THT:TO-92_Inline, F.Cu at (399.2, 87.6)
- added R18: 0, Resistor_SMD:R_0603_1608Metric, F.Cu at (135.3, 144.5)
- added R19: 0, Resistor_SMD:R_0603_1608Metric, F.Cu at (135.3, 147.0)
- added R20: 5 MΩ, Resistor_SMD:R_0402_1005Metric, F.Cu at (100.7, 157.2)
- added R21: 10k, Resistor_SMD:R_0402_1005Metric, F.Cu at (94.9, 153.2)
- added R22: 10k, Resistor_SMD:R_0402_1005Metric, F.Cu at (94.9, 155.2)
- added R23: 200, Resistor_SMD:R_0402_1005Metric, F.Cu at (94.9, 157.2)
- added R24: 4.7k, Resistor_SMD:R_0402_1005Metric, F.Cu at (357.7, 89.0)
- added R27: 0, Resistor_SMD:R_0603_1608Metric, F.Cu at (395.2, 89.8)
- added R28: 10k, Resistor_SMD:R_0402_1005Metric, F.Cu at (357.7, 93.0)
- added R29: 10k, Resistor_SMD:R_0402_1005Metric, F.Cu at (357.7, 95.0)
- added R30: 47, Resistor_SMD:R_0402_1005Metric, F.Cu at (360.6, 89.0)
- added R31: 47, Resistor_SMD:R_0402_1005Metric, F.Cu at (360.6, 91.0)
- added R32: 200, Resistor_SMD:R_0402_1005Metric, F.Cu at (360.6, 93.0)
- added R33: 0.05 1%, Resistor_SMD:R_2512_6332Metric, F.Cu at (379.1, 116.5)
- added R34: 10, Resistor_SMD:R_0402_1005Metric, F.Cu at (376.1, 128.5)
- added R35: 10, Resistor_SMD:R_0402_1005Metric, F.Cu at (376.1, 130.4)
- added R36: 10k, Resistor_SMD:R_0402_1005Metric, F.Cu at (376.1, 132.4)
- added R37: 350, Resistor_SMD:R_0402_1005Metric, F.Cu at (376.1, 122.5)
- added R38: 5.1k 1%, Resistor_SMD:R_0402_1005Metric, F.Cu at (213.5, 105.3)
- added R39: 5.1k 1%, Resistor_SMD:R_0402_1005Metric, F.Cu at (213.5, 101.8)
- added R48: 0, Resistor_SMD:R_0402_1005Metric, F.Cu at (392.6, 104.9)
- added R49: 5.1k, Resistor_SMD:R_0402_1005Metric, F.Cu at (392.6, 106.9)
- added R50: 1k, Resistor_SMD:R_0402_1005Metric, F.Cu at (392.6, 108.9)
- added R51: 1.5k, Resistor_SMD:R_0402_1005Metric, F.Cu at (392.6, 110.9)
- added TP1: BOOT, TestPoint:TestPoint_Bridge_Pitch2.54mm_Drill0.7mm, F.Cu at (129.1, 142.4)
- added TP10: VBUS, Connector_PinSocket_2.54mm:PinSocket_1x01_P2.54mm_Vertical, F.Cu at (214.0, 110.8)
- added TP2: DTR, TestPoint:TestPoint_Bridge_Pitch2.54mm_Drill0.7mm, F.Cu at (389.0, 97.5)
- added TP3: RTS, TestPoint:TestPoint_Bridge_Pitch2.54mm_Drill0.7mm, F.Cu at (389.0, 94.1)
- added TP4: LOOP_OUT_3, TestPoint:TestPoint_Bridge_Pitch2.54mm_Drill0.7mm, F.Cu at (389.0, 90.6)
- added TP5: LOOP_OUT_2, TestPoint:TestPoint_Bridge_Pitch2.54mm_Drill0.7mm, F.Cu at (389.0, 87.2)
- added TP6: LOOP_OUT_1, TestPoint:TestPoint_Bridge_Pitch2.54mm_Drill0.7mm, F.Cu at (389.0, 83.7)
- added TP7: VBUSunreg, TestPoint:TestPoint_Bridge_Pitch2.54mm_Drill0.7mm, F.Cu at (363.0, 119.2)
- added TP8: LOOP_OUT_2, TestPoint:TestPoint_Bridge_Pitch2.54mm_Drill0.7mm, F.Cu at (363.0, 115.8)
- added TP9: 3V3, TestPoint:TestPoint_Bridge_Pitch2.54mm_Drill0.7mm, F.Cu at (363.0, 122.7)
- added U2: ESP32-WROOM-32UE, RF_Module:ESP32-WROOM-32UE, F.Cu at (182.3, 57.6)
- added U5: INA226, Package_SO:TSSOP-10_3x3mm_P0.5mm, F.Cu at (381.2, 128.7)
- added U6: MAX40200AUK, Package_TO_SOT_SMD:SOT-23-5, F.Cu at (202.6, 110.8)
- added U9: 74LVC3G17V8-7, easyeda2kicad:VSSOP-8_L2.1-W2.4-P0.50-LS3.2-BL, F.Cu at (395.7, 106.4)
- added Y1: 32.768kHz 7pF, Crystal:Crystal_SMD_2012-2Pin_2.0x1.2mm_HandSoldering, F.Cu at (95.7, 159.8)
- C1: value 10uF -> 100nF; moved to F.Cu
- C10, C11: value 22uF -> 100nF; footprint Capacitor_SMD:C_0805_2012Metric -> Capacitor_SMD:C_0402_1005Metric; moved to F.Cu
- C12, H3, H4, R1: moved to F.Cu
- C13, C14: value 1nF -> 10uF; footprint Capacitor_THT:C_Radial_D5.0mm_H11.0mm_P2.00mm -> Capacitor_SMD:C_0402_1005Metric; moved to F.Cu
- C2, C5: value 100nF -> 10uF; moved to F.Cu
- C23: value 250nF -> 100nF; footprint Capacitor_THT:C_Radial_D5.0mm_H11.0mm_P2.00mm -> Capacitor_SMD:C_0402_1005Metric; moved to F.Cu
- C24: value 250nF -> 10uF; footprint Capacitor_THT:C_Radial_D5.0mm_H11.0mm_P2.00mm -> Capacitor_SMD:C_0402_1005Metric; moved to F.Cu
- C3: value 1uF -> 10uF; moved to F.Cu
- C4: value 10uF -> 1uF; moved to F.Cu
- C7: value 10uF -> 22uF >10v XR5; footprint Capacitor_SMD:C_0402_1005Metric -> Capacitor_SMD:C_0805_2012Metric; moved to F.Cu
- J2: value Conn_01x10_Socket -> UART; footprint Connector_PinSocket_2.54mm:PinSocket_1x10_P2.54mm_Horizontal -> Connector_PinSocket_2.54mm:PinSocket_1x04_P2.54mm_Horizontal; moved to F.Cu
- J3: value USB-C Receptacle -> I2C; footprint Connector_USB:USB_C_Receptacle_G-Switch_GT-USB-7010ASV -> Connector_PinSocket_2.54mm:PinSocket_1x04_P2.54mm_Horizontal; moved to F.Cu
- J6: renamed from J4; moved to F.Cu
- R2, R5: value 10k -> 50
- R25: value 5.1k 1% -> 4.7k; moved to F.Cu
- R26: value 5.1k 1% -> 0; footprint Resistor_SMD:R_0402_1005Metric -> Resistor_SMD:R_0603_1608Metric; moved to F.Cu
- R4, R6: value 22 -> 50
- R42: renamed from R29; value 5k -> 5.1k
- R43: renamed from R30; value 5k -> 5.1k
- U10: renamed from U7; value TLC555xD -> TLC555CDR
- U3: value TLV76133DCY -> CH340K; footprint Package_TO_SOT_SMD:SOT-223-3_TabPin2 -> Package_SO:SSOP-10-1EP_3.9x4.9mm_P1mm_EP2.1x3.3mm; moved to F.Cu
- U4: value MAX40200AUK -> TLV76133DCY; footprint Package_TO_SOT_SMD:SOT-23-5 -> Package_TO_SOT_SMD:SOT-223-3_TabPin2; moved to F.Cu
- U7: renamed from U5; value TLC555xD -> TLC555CDR
- U8: renamed from U6; value TLC555xD -> TLC555CDR
- moved H4 233.9 mm to (68.0, 25.0), turned to 0 degrees
- moved R26 208.8 mm to (395.2, 87.3)
- moved C11 204.9 mm to (397.5, 100.0), turned to 0 degrees
- moved C14 204.6 mm to (400.4, 96.0), turned to 0 degrees
- moved C10 201.4 mm to (397.5, 98.0), turned to 0 degrees
- moved C13 198.3 mm to (400.4, 94.0), turned to 0 degrees
- moved C12 197.4 mm to (400.4, 92.1), turned to 0 degrees
- moved AE1 180.0 mm to (81.0, 42.0)
- moved R25 171.7 mm to (357.7, 91.0)
- moved R45 166.5 mm to (335.2, 26.3)
- moved R46 166.5 mm to (334.0, 27.3)
- moved R47 166.5 mm to (328.7, 27.6)
- moved R6 166.5 mm to (329.0, 25.5)
- moved R15 166.5 mm to (320.3, 28.8)
- moved R16 166.5 mm to (320.3, 26.3)
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- renumbered C15 to C25, C16 to C26, C17 to C27, C18 to C28, C19 to C29, C20 to C30, C21 to C31, C22 to C32, C26 to C33, C27 to C34, C28 to C35, C29 to C36, D1 to D2, D3 to D4, J5 to J7, JP4 to JP1, JP5 to JP2, JP6 to JP3, JP7 to JP4, JP8 to JP7, JP9 to JP8, R17 to R10, R18 to R11, R19 to R12, R20 to R13, R21 to R14, R22 to R15, R23 to R16, R24 to R17, R9 to R2, R10 to R3, R11 to R4, R27 to R40, R28 to R41, R31 to R44, R32 to R45, R33 to R46, R34 to R47, R12 to R5, R13 to R6, R14 to R7, R15 to R8, R16 to R9, TP2 to TP11, TP3 to TP12, TP4 to TP13, TP5 to TP14, TP6 to TP15, TP7 to TP16, TP8 to TP17, TP9 to TP18, TP10 to TP19, TP11 to TP20, TP12 to TP21, TP13 to TP22, U2 to U1
Connections:
- C11 pad 1: +3.3V -> GND
- C11 pad 2: GND -> Net-(C11-Pad2)
- C12 pad 2: /VBUS_{fused} -> Net-(C12-Pad2)
- C13 pad 1: Net-(JP4-B) -> VBUS_{unregulated}
- C14 pad 1: Net-(JP5-B) -> +3.3V
- C23 pad 1: Net-(JP4-B) -> GND
- C23 pad 2: Net-(JP6-B) -> /Power Interface/VBUS_{fused}
- C24 pad 1: Net-(JP5-B) -> VBUS_{unregulated}
- C24 pad 2: Net-(JP7-B) (its old number) -> GND
- C27 pad 1: Net-(JP4-B) -> Net-(JP1-B)
- C28 pad 1: Net-(JP5-B) -> Net-(JP2-B)
- C29 pad 2: +5V -> /Inductive Loop/VBUS_SENSOR_IN
- C3 pad 2: /EN -> +3.3V
- C30 pad 2: +5V -> /Inductive Loop/VBUS_SENSOR_IN
- C31 pad 2: +5V -> /Inductive Loop/VBUS_SENSOR_IN
- C32 pad 2: +5V -> /Inductive Loop/VBUS_SENSOR_IN
- C35 pad 2: +5V -> /Inductive Loop/VBUS_SENSOR_IN
- C36 pad 2: +5V -> /Inductive Loop/VBUS_SENSOR_IN
- C4 pad 1: GND -> /EN
- C4 pad 2: +3.3V -> GND
- C7 pad 1: VBUS_{unregulated} -> +3.3V
- D2 pad 1: Net-(D1-K) -> Net-(D2-K)
- D4 pad 1: Net-(D3-K) (its old number) -> Net-(D4-K)
- J2 pad 1: Net-(J2-Pin_1) -> +3.3V
- J2 pad 2: Net-(J2-Pin_2) -> /TXD0_GPIO_1
- J2 pad 3: Net-(J2-Pin_3) -> /RXD0_GPIO_3
- J2 pad 4: Net-(J2-Pin_4) -> GND
- J6 pad 1: /VBUS_{fused} -> /GPIO_14
- J6 pad 2: GND -> /GPIO_19
- J6 pad 3: /GPIO_4 -> /GPIO_23
- J6 pad 4: /GPIO_10 -> /GPIO_25
- J6 pad 5: /TXD0 -> /GPIO_26
- J6 pad 6: /RXD0 -> /GPIO_34
- J6 pad 7: GND -> /GPIO_35
- JP1 pad 2: Net-(JP4-B) -> Net-(JP1-B)
- JP2 pad 2: Net-(JP5-B) -> Net-(JP2-B)
- JP3 pad 2: Net-(JP6-B) -> Net-(JP3-B)
- JP4 pad 2: Net-(JP7-B) (its old number) -> Net-(JP4-B)
- R10 pad 2: Net-(J2-Pin_6) -> Net-(J4-Pin_6)
- R11 pad 2: Net-(J2-Pin_7) -> Net-(J4-Pin_7)
- R12 pad 2: Net-(J2-Pin_8) -> Net-(J4-Pin_13)
- R13 pad 2: Net-(J2-Pin_9) -> Net-(J4-Pin_12)
- R14 pad 2: Net-(J2-Pin_10) -> Net-(J4-Pin_11)
- R15 pad 2: unconnected-(R22-Pad2) -> Net-(J4-Pin_10)
- R16 pad 2: unconnected-(R23-Pad2) -> Net-(J4-Pin_9)
- R17 pad 2: unconnected-(R24-Pad2) -> Net-(J4-Pin_8)
- R2 pad 1: +3.3V -> Net-(U1-LED0)
- R2 pad 2: /GPIO_8 -> Net-(D2-K)
- R2 pad 1: Net-(U2-LED0) -> Net-(U1-LED0)
- R2 pad 2: Net-(D1-K) -> Net-(D2-K)
- R25 pad 1: GND -> +3.3V
- R25 pad 2: Net-(J3-CC1) -> /SCL_GPIO_22
- R26 pad 1: GND -> USB D+
- R26 pad 2: Net-(J3-CC2) -> Net-(U3-UD+)
- R4 pad 1: /USB D- -> Net-(U1-LED2)
- R4 pad 2: Net-(U1-IO18) -> Net-(D4-K)
- R4 pad 1: Net-(U2-LED2) -> Net-(U1-LED2)
- R4 pad 2: Net-(D3-K) (its old number) -> Net-(D4-K)
- R40 pad 2: Net-(JP6-B) -> Net-(JP3-B)
- R41 pad 2: Net-(JP7-B) (its old number) -> Net-(JP4-B)
- R42 pad 1: +5V -> Net-(JP5-A)
- R43 pad 1: +5V -> Net-(JP6-A)
- R5 pad 1: +3.3V -> Net-(U1-LED3)
- R5 pad 2: Net-(U1-IO2) -> Net-(J4-Pin_1)
- R5 pad 1: Net-(U2-LED3) -> Net-(U1-LED3)
- R5 pad 2: Net-(J2-Pin_1) -> Net-(J4-Pin_1)
- R6 pad 1: Net-(U1-IO19) -> Net-(U1-LED4)
- R6 pad 2: /USB D+ -> Net-(J4-Pin_2)
- R6 pad 1: Net-(U2-LED4) -> Net-(U1-LED4)
- R6 pad 2: Net-(J2-Pin_2) -> Net-(J4-Pin_2)
- R7 pad 2: Net-(J2-Pin_3) -> Net-(J4-Pin_3)
- R8 pad 2: Net-(J2-Pin_4) -> Net-(J4-Pin_4)
- R9 pad 2: Net-(J2-Pin_5) -> Net-(J4-Pin_5)
- RV1 pad 3: +5V -> /Inductive Loop/VBUS_SENSOR_IN
- RV2 pad 3: +5V -> /Inductive Loop/VBUS_SENSOR_IN
- RV3 pad 3: +5V -> /Inductive Loop/VBUS_SENSOR_IN
- SW1 pad 1: Net-(C6-Pad2) -> Net-(C11-Pad2)
- SW2 pad 1: Net-(R8-Pad2) -> Net-(C12-Pad2)
- U1 pad 10: Net-(U2-LED4) -> Net-(U1-LED4)
- U1 pad 23: /GPIO_8 -> GND
- U1 pad 26: /GPIO_3 -> /SCL_GPIO_22
- U1 pad 27: /GPIO_1 -> /SDA_GPIO_21
- U1 pad 6: Net-(U2-LED0) -> Net-(U1-LED0)
- U1 pad 8: Net-(U2-LED2) -> Net-(U1-LED2)
- U1 pad 9: Net-(U2-LED3) -> Net-(U1-LED3)
- U10 pad 4: +5V -> /Inductive Loop/VBUS_SENSOR_IN
- U10 pad 8: +5V -> /Inductive Loop/VBUS_SENSOR_IN
- U3 pad 1: GND -> Net-(U3-UD+)
- U3 pad 2: +3.3V -> Net-(U3-UD-)
- U3 pad 3: VBUS_{unregulated} -> GND
- U4 pad 1: /VBUS_{fused} -> GND
- U4 pad 2: GND -> Net-(U4-VO)
- U4 pad 3: /VBUS_{fused} -> VBUS_{unregulated}
- U7 pad 2: Net-(JP4-B) -> Net-(JP1-B)
- U7 pad 4: +5V -> /Inductive Loop/VBUS_SENSOR_IN
- U7 pad 6: Net-(JP4-B) -> Net-(JP1-B)
- U7 pad 8: +5V -> /Inductive Loop/VBUS_SENSOR_IN
- U8 pad 2: Net-(JP5-B) -> Net-(JP2-B)
- U8 pad 4: +5V -> /Inductive Loop/VBUS_SENSOR_IN
- U8 pad 6: Net-(JP5-B) -> Net-(JP2-B)
- U8 pad 8: +5V -> /Inductive Loop/VBUS_SENSOR_IN
Routing:
- net unconnected-(R24-Pad2): vias 1 -> 0
- net unconnected-(R23-Pad2): vias 1 -> 0
- net VBUS_{unregulated}: vias 3 -> 0
- net Net-(U8-DIS): vias 2 -> 0
- net Net-(U7-DIS): vias 5 -> 0
- net Net-(U2-LED0): vias 2 -> 0
- net Net-(U10-DIS): vias 1 -> 0
- net Net-(U10-CV): vias 1 -> 0
- net Net-(U1-LED15): vias 2 -> 0
- net Net-(U1-LED14): vias 2 -> 0
- net Net-(U1-LED12): vias 2 -> 0
- net Net-(U1-LED11): vias 2 -> 0
- net Net-(U1-LED1): vias 1 -> 0
- net Net-(U1-IO2): vias 3 -> 0
- net Net-(U1-IO19): vias 1 -> 0
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Other:
- board size 100 x 100 mm -> 165.5 x 100.5 mm
- board text added: "v0.5"
- board text removed: "v0.4"
