File: kicad/IntelligentTrafficLight.kicad_sch (KiCad schematic)
At the start: 61 parts, among them J1 USB-C Receptacle, J2 Conn_01x07_Socket, J3 Conn_01x10_Socket, J4 Conn_01x07_Socket, J5 Conn_01x03_Pin, SW1 Pushbutton, SW3 Pushbutton, U1 ESP32-C3-MINI-1-H4X, U2 TLV76133DCY, U3 PCA9685PW

Commit message: add comments to kicad schematic
Parts:
- added U4: MAX40200AUK, Package_TO_SOT_SMD:SOT-23-5, symbol Analog_Switch:MAX40200AUK
- renumbered C32 to C1, C36 to C10, C37 to C11, C9 to C12, C6 to C2, C33 to C3, C10 to C4, C31 to C5, C34 to C6, C4 to C7, C5 to C8, C35 to C9, D3 to D2, D4 to D3, D2 to D4, H4 to H1, H3 to H2, H2 to H3, H1 to H4, J5 to J1, J3 to J2, J1 to J3, J2 to J5, JP7 to JP1, JP8 to JP2, JP9 to JP3, R35 to R1, R20 to R10, R21 to R11, R22 to R12, R23 to R13, R24 to R14, R25 to R15, R26 to R16, R27 to R17, R28 to R18, R29 to R19, R39 to R2, R30 to R20, R31 to R21, R32 to R22, R33 to R23, R34 to R24, R7 to R25, R8 to R26, R6 to R3, R37 to R4, R38 to R5, R36 to R6, R40 to R7, R41 to R8, SW3 to SW1, SW1 to SW2, U3 to U2, U2 to U3
Connections:
- net +5V: now also U4.5 (OUT); no longer C12.2, D4.6 (VCC), F1.1, J4.1 (Pin_1)
- net GND: now also U4.2 (GND)
- new net VBUS_{fused}: C12.2, D4.6 (VCC), F1.1, J4.1 (Pin_1), U4.1 (VDD), U4.3 (EN)
Other:
- note added: "USB Backfeed Protection"
- moved on the sheet: C6, C7, C8, R7, SW1, U3

Commit message: small pcb change
Parts:
- removed C1, C4: 10uF, Capacitor_SMD:C_0402_1005Metric, symbol Device:C
- removed JP1, JP2, JP3: SolderJumper_2_Open, Jumper:SolderJumper-2_P1.3mm_Open_RoundedPad1.0x1.5mm, symbol Jumper:SolderJumper_2_Open
- removed R2: 10k, Resistor_SMD:R_0402_1005Metric, symbol Device:R
- added C1, C4: 10uF, Capacitor_SMD:C_0402_1005Metric, symbol Device:C_Small
- added C31, C33: 4.7uF, Capacitor_SMD:C_0402_1005Metric, symbol Device:C_Small
- added D5: TT0314TPX, easyeda2kicad:DFN2510-10_L2.5-W1.0-P0.50-BL, symbol EASYEDA2KICAD:TT0314TPX
- added U8, U9: MX5052SL, easyeda2kicad:SOP-8_L5.1-W3.9-P1.27-LS6.0-BL, symbol EASYEDA2KICAD:MX5052SL
- C2: value 100nF -> 10uF
- C5: value 100nF -> 1uF
- C7, C8: Voltage Rating (none) -> >6.3v
Connections:
- net +5V is gone; now on net VBUS_{unregulated}: U4.5 (OUT)
- net GPIO_5 is gone; now on net LOOP_OUT_1: U1.19 (IO5)
- net GPIO_6 is gone; now on net LOOP_OUT_2: U1.20 (IO6)
- net GPIO_7 is gone; now on net LOOP_OUT_3: U1.21 (IO7)
- net +3.3V: now also C31.1, C4.2, U8.5 (OUT), U8.6 (OUT), U8.7 (OUT), U8.8 (OUT); no longer C5.2
- net GND: now also C5.2, C1.2, C31.2, C33.2, C4.1, D5.3 (GND), D5.8 (GND), U8.2 (GND), U9.2 (GND), U9.3 (IN), U9.4 (IN); no longer C5.1
- net GPIO_0: now also D5.2 (I/O_2), U8.3 (IN), U8.4 (IN), U9.5 (OUT), U9.6 (OUT), U9.7 (OUT), U9.8 (OUT)
- net VBUS_{fused}: now also C5.1
- net VBUS_{unregulated}: now also C1.1, C33.1, U8.1 (VS), U9.1 (VS)
- no-connect marks 30 -> 37
Other:
- note added: "GPIO_0 protected with 100Ω and 30mA polyfuse"
- note added: "Ideal Diode Vf - 40mV"
- note added: "TVS Diode 3.5V Clamping 3.3V Vrwm"
- note removed: "this usb-c receptacle is so horrible - pls replace"
- moved on the sheet: C7, C8, F1, H1, H2, H3, H4, J3, J4, J5, R1, R25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

Commit message: update!
Parts:
- removed C1, C2: 10uF, Capacitor_SMD:C_0402_1005Metric, symbol Device:C_Small
- removed C10, C11, C9: 22uF, Capacitor_SMD:C_0805_2012Metric, symbol Device:C
- removed C12: 100nF, Capacitor_SMD:C_0402_1005Metric, symbol Device:C_Small
- removed C3, C5: 1uF, Capacitor_SMD:C_0402_1005Metric, symbol Device:C_Small
- removed C7, C8: 10uF, Capacitor_SMD:C_0402_1005Metric, symbol Device:C
- removed D4: TPD3E001DRYR, Package_SON:Texas_USON-6_1x1.45mm_P0.5mm_SMD, symbol EasyEDA:TPD3E001DRYR
- removed D5: TT0314TPX, easyeda2kicad:DFN2510-10_L2.5-W1.0-P0.50-BL, symbol EASYEDA2KICAD:TT0314TPX
- removed F1: 1.5A, Fuse:Fuse_1206_3216Metric_Pad1.42x1.75mm_HandSolder, symbol Device:Polyfuse
- removed H1, H2, H3, H4: MountingHole_Pad, MountingHole:MountingHole_3.2mm_M3_Pad, symbol Mechanical:MountingHole_Pad
- removed J3: USB-C Receptacle, Connector_USB:USB_C_Receptacle_G-Switch_GT-USB-7010ASV, symbol Connector:USB_C_Receptacle_USB2.0_16P
- removed R1: 10k, Resistor_SMD:R_0402_1005Metric, symbol Device:R
- removed R25, R26: 5.1k 1%, Resistor_SMD:R_0402_1005Metric, symbol Device:R
- removed R3: 10k, Resistor_SMD:R_0402_1005Metric, symbol Device:R_Small
- removed R6: 22, Resistor_SMD:R_0402_1005Metric, symbol Device:R_Small
- removed TP1: VBUS, Connector_PinSocket_2.54mm:PinSocket_1x01_P2.54mm_Vertical, symbol Connector:TestPoint
- removed U1: ESP32-C3-MINI-1-H4X, EASYEDA2KICAD:WIFIM-SMD_ESP32-C3-MINI-1, symbol EASYEDA2KICAD:ESP32-C3-MINI-1-H4X
- removed U3: TLV76133DCY, Package_TO_SOT_SMD:SOT-223-3_TabPin2, symbol Regulator_Linear:TLV76133DCY
- removed U4: MAX40200AUK, Package_TO_SOT_SMD:SOT-23-5, symbol Analog_Switch:MAX40200AUK
- removed U8, U9: MX5052SL, easyeda2kicad:SOP-8_L5.1-W3.9-P1.27-LS6.0-BL, symbol EASYEDA2KICAD:MX5052SL
- added C32: 1uF, Capacitor_SMD:C_0402_1005Metric, symbol Device:C_Small
- added C34: 22uF >10v XR5, Capacitor_SMD:C_0805_2012Metric, symbol Device:C
- added C35, C36, C37: 100nF, Capacitor_SMD:C_0402_1005Metric, symbol Device:C_Small
- added D5, D8: LED, LED_THT:LED_D5.0mm, symbol Device:LED
- added FB1: FerriteBead R600, Inductor_SMD:L_0603_1608Metric, symbol Device:FerriteBead
- added J6: UART, symbol Connector:Conn_01x04_Socket
- added J7: I2C, symbol Connector:Conn_01x04_Socket
- added Q1, Q2: S8050, Package_TO_SOT_THT:TO-92_Inline, symbol Transistor_BJT:S8050
- added R1: 4.7k, Resistor_SMD:R_0402_1005Metric, symbol Device:R_Small
- added R2, R3, R39, R40: 10k, Resistor_SMD:R_0402_1005Metric, symbol Device:R
- added R26, R45: 200, Resistor_SMD:R_0402_1005Metric, symbol Device:R_Small
- added R41, R42: 0, Resistor_SMD:R_0603_1608Metric, symbol Device:R_Small
- added TP16, TP17: TestPoint_2Pole, TestPoint:TestPoint_Bridge_Pitch3.81mm_Drill1.3mm, symbol Connector:TestPoint_2Pole
- added U10: ESP32-WROOM-32UE, RF_Module:ESP32-WROOM-32UE, symbol RF_Module:ESP32-WROOM-32UE
- added U11: CH340K, Package_SO:SSOP-10-1EP_3.9x4.9mm_P1mm_EP2.1x3.3mm, symbol Interface_USB:CH340K
- R4: value 22 -> 4.7k
- R7, R8: value 0 -> 47
Connections:
- net GPIO_3 is gone; now on net SCL/GPIO_22: U2.26 (SCL)
- net GPIO_8 is gone; now on net GND: U2.23 (~{OE})
- net +3.3V: now also R4.1, C34.1, C35.1, C37.1, J6.1 (Pin_1), J7.1 (Pin_1), R1.1, R3.2, R39.1, U10.2 (VDD), U11.10 (V3), U11.7 (VCC); no longer R5.1
- net EN: now also C32.1, Q1.3 (C), R39.2, U10.3 (EN)
- net GND: now also R5.2, C32.2, C34.2, C35.2, C36.1, C37.2, D5.1 (K), D8.1 (K), J6.4 (Pin_4), J7.4 (Pin_4), U10.1 (GND), U10.15 (GND), U10.38 (GND), U10.39 (GND), U11.11 (GND), U11.3 (GND); no longer J4.2 (Pin_2), J4.7 (Pin_7)
- net GPIO_0: now also Q2.3 (C), R3.1, R45.2, U10.25 (IO0)
- net LOOP_OUT_1: now also U10.11 (IO26)
- net LOOP_OUT_2: now also U10.26 (IO4)
- net LOOP_OUT_3: now also U10.10 (IO25)
- net RXD0: now also J6.3 (Pin_3), U10.34 (RXD0/IO3), U11.8 (TXD); no longer J4.6 (Pin_6)
- net TXD0: now also J6.2 (Pin_2), U10.35 (TXD0/IO1), U11.9 (RXD); no longer J4.5 (Pin_5)
- net USB D+: now also TP16.1
- net USB D-: now also TP17.1; no longer R4.1
- net VBUS_{unregulated}: now also FB1.1
- net at R8.2, SW2.1: now also C36.2
- net SCL/GPIO_22: now reaches R4.2
- net SCL/GPIO_22: now also J7.3 (Pin_3), U10.36 (IO22)
- net GPIO_1 renamed SDA/GPIO_21
- net SDA/GPIO_21: now also J7.2 (Pin_2), R1.2, U10.33 (IO21)
- net GPIO_10 renamed GPIO_16
- net GPIO_16: now also U10.27 (IO16)
- net GPIO_4 renamed GPIO_15
- net GPIO_15: now also U10.23 (IO15)
- net VBUS_{fused} renamed GPIO_13
- net GPIO_13: now also U10.16 (IO13)
- new net: Q2.1 (E), R2.1, U11.4 (~{DTR})
- new net: Q2.2 (B), R40.2
- new net: Q1.1 (E), R40.1, U11.6 (~{RTS})
- new net: R42.1, TP17.2
- new net: R42.2, U11.2 (UD-)
- new net: Q1.2 (B), R2.2
- new net: R5.1, U10.14 (IO12)
- new net: D8.2 (A), R45.1
- new net: D5.2 (A), R26.1
- new net: R41.1, TP16.2
- new net: R41.2, U11.1 (UD+)
- new net GPIO_14: J4.2 (Pin_2), U10.13 (IO14)
- new net GPIO_17: J4.5 (Pin_5), U10.28 (IO17)
- new net GPIO_18: J4.6 (Pin_6), U10.30 (IO18)
- new net GPIO_19: J4.7 (Pin_7), U10.31 (IO19)
- new net GPIO_23: U10.37 (IO23)
- new net GPIO_32: U10.8 (IO32)
- new net GPIO_33: U10.9 (IO33)
- new net GPIO_34: U10.6 (IO34)
- new net GPIO_35: U10.7 (IO35)
- new net Inductive Loop/VBUS_SENSOR_IN: FB1.2
- new net LED/GPIO_27: R26.2, U10.12 (IO27)
- new net SENSOR_VN: U10.5 (SENSOR_VN)
- new net SENSOR_VP: U10.4 (SENSOR_VP)
- no-connect marks 37 -> 14
Other:
- added sheet Power Interface (Power_Interface.kicad_sch)
- sheet Inductive Loop ports: added VBUS_SENSOR_IN; removed none
- note added: "CH340K USB to UART"
- note added: "ESP32-WROOM-32UE"
- note removed: "3v3 LDO"
- note removed: "ESD Protection"
- note removed: "GPIO_0 protected with 100Ω and 30mA polyfuse"
- note removed: "Ideal Diode Vf - 40mV"
- note removed: "TVS Diode 3.5V Clamping 3.3V Vrwm"
- note removed: "USB Backfeed Protection"
- moved on the sheet: C31, C33, C4, C6, D1, D2, D3, J1, J2, J4, J5, R10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

Commit message: more updates
Parts:
- removed J2: Conn_01x10_Socket, Connector_PinSocket_2.54mm:PinSocket_1x10_P2.54mm_Horizontal, symbol Connector:Conn_01x10_Socket
- removed R3: 10k, Resistor_SMD:R_0402_1005Metric, symbol Device:R
- removed TP16, TP17: TestPoint_2Pole, TestPoint:TestPoint_Bridge_Pitch3.81mm_Drill1.3mm, symbol Connector:TestPoint_2Pole
- added C1: 100nF, Capacitor_SMD:C_0402_1005Metric, symbol Device:C_Small
- added C2: 10uF, symbol Device:C_Small
- added C3: 10uF, Capacitor_SMD:C_0402_1005Metric, symbol Device:C_Small
- added C8, C9: 12pF/50V, symbol Device:C_Small
- added D5: TT0314TPX, easyeda2kicad:DFN2510-10_L2.5-W1.0-P0.50-BL, symbol EASYEDA2KICAD:TT0314TPX
- added J1: JTAG ESP-Prog, symbol Connector:Conn_01x10_Socket
- added J4: Conn_02x07_Top_Bottom, symbol Connector_Generic:Conn_02x07_Top_Bottom
- added R18, R19: 0, Resistor_SMD:R_0603_1608Metric, symbol Device:R_Small
- added R20: 10k, Resistor_SMD:R_0402_1005Metric, symbol Device:R
- added TP1: BOOT, TestPoint:TestPoint_Bridge_Pitch2.54mm_Drill0.7mm, symbol Connector:TestPoint
- added TP2: DTR, TestPoint:TestPoint_Bridge_Pitch2.54mm_Drill0.7mm, symbol Connector:TestPoint_2Pole
- added TP3: RTS, TestPoint:TestPoint_Bridge_Pitch2.54mm_Drill0.7mm, symbol Connector:TestPoint_2Pole
- added TP4: LOOP_OUT_3, TestPoint:TestPoint_Bridge_Pitch2.54mm_Drill0.7mm, symbol Connector:TestPoint_2Pole
- added TP5: LOOP_OUT_2, TestPoint:TestPoint_Bridge_Pitch2.54mm_Drill0.7mm, symbol Connector:TestPoint_2Pole
- added TP6: LOOP_OUT_1, TestPoint:TestPoint_Bridge_Pitch2.54mm_Drill0.7mm, symbol Connector:TestPoint_2Pole
- added Y1: 32.768kHz, symbol Device:Crystal
- C13: renamed from C33; value 4.7uF -> 10uF
- C14: renamed from C31; value 4.7uF -> 10uF
- renumbered C37 to C10, C6 to C11, C36 to C12, C32 to C4, C4 to C5, C35 to C6, C34 to C7, D5 to D1, D1 to D2, D2 to D3, D3 to D4, D8 to D6, J6 to J2, J7 to J3, J1 to J5, J4 to J6, J5 to J7, R39 to R1, R17 to R10, R18 to R11, R19 to R12, R20 to R13, R21 to R14, R22 to R15, R23 to R16, R24 to R17, R9 to R2, R5 to R21, R26 to R22, R1 to R23, R4 to R24, R41 to R25, R42 to R26, R2 to R27, R40 to R28, R7 to R29, R10 to R3, R8 to R30, R45 to R31, R11 to R4, R12 to R5, R13 to R6, R14 to R7, R15 to R8, R16 to R9, U2 to U1, U10 to U2, U11 to U3
Connections:
- net +3.3V: now also C1.1, C2.1, C3.2, J1.10 (Pin_10), R20.2
- net EN: now also J1.1 (Pin_1)
- net GND: now also C1.2, C2.2, C3.1, C8.2, C9.2, D5.3 (GND), D5.8 (GND), J1.2 (Pin_2), J1.6 (Pin_6), J1.8 (Pin_8), J4.14 (Pin_14)
- net GPIO_14: now also J6.1 (Pin_1), U2.26 (IO4); no longer J6.2 (Pin_2), U2.13 (IO14)
- net GPIO_19: now also J6.2 (Pin_2); no longer J6.7 (Pin_7)
- net GPIO_23: now also J6.3 (Pin_3)
- net GPIO_34: now also J6.6 (Pin_6)
- net GPIO_35: now also J6.7 (Pin_7)
- net LOOP_OUT_1: now also U2.27 (IO16), TP6.2; no longer U2.11 (IO26)
- net LOOP_OUT_2: now also U2.28 (IO17), TP5.2; no longer U2.26 (IO4)
- net LOOP_OUT_3: now also U2.30 (IO18), TP4.2; no longer U2.10 (IO25)
- net USB D+: now also R25.1
- net USB D-: now also R26.1
- net at Q2.1 (E), R27.1, U3.4 (~{DTR}): now also TP2.1, TP2.2
- net at R16.2: now also J4.9 (Pin_9)
- net at Q1.1 (E), R28.1, U3.6 (~{RTS}): now also TP3.1, TP3.2
- net at R9.2: now also J4.5 (Pin_5)
- net at R6.2: now also J4.2 (Pin_2)
- net at R5.2: now also J4.1 (Pin_1)
- net at R7.2: now also J4.3 (Pin_3)
- net at R8.2: now also J4.4 (Pin_4)
- net at R13.2: now also J4.12 (Pin_12)
- net at R10.2: now also J4.6 (Pin_6)
- net TDI_GPIO_12: now reaches R21.1, U2.14 (IO12)
- net TDI_GPIO_12: now also J1.3 (Pin_3)
- net at R12.2: now also J4.13 (Pin_13)
- net at R17.2: now also J4.8 (Pin_8)
- net at R14.2: now also J4.11 (Pin_11)
- net at R11.2: now also J4.7 (Pin_7)
- net at R15.2: now also J4.10 (Pin_10)
- net GPIO_0 renamed BOOT_GPIO_0
- net BOOT_GPIO_0: now also R20.1, TP1.1
- net GPIO_13 renamed TCK_GPIO_13
- net TCK_GPIO_13: now also J1.7 (Pin_7); no longer J6.1 (Pin_1)
- net GPIO_15 renamed TDO_GPIO_15
- net TDO_GPIO_15: now also J1.5 (Pin_5); no longer J6.3 (Pin_3)
- net GPIO_16 renamed GPIO_25
- net GPIO_25: now also U2.10 (IO25); no longer U2.27 (IO16)
- net GPIO_17 renamed GPIO_26
- net GPIO_26: now also U2.11 (IO26); no longer U2.28 (IO17)
- removed net GPIO_18: J6.6 (Pin_6), U2.30 (IO18)
- net GPIO_32: no longer names the net of U2.8 (IO32)
- net GPIO_32: now also R19.2
- net GPIO_33: no longer names the net of U2.9 (IO33)
- net GPIO_33: now also R18.2
- net LED/GPIO_27 renamed LED_GPIO_27
- net RXD0 renamed RXD0_GPIO_3
- net RXD0_GPIO_3: now also D5.4 (I/O_3)
- net SCL/GPIO_22 renamed SCL_GPIO_22
- net SCL_GPIO_22: now also D5.2 (I/O_2)
- net SDA/GPIO_21 renamed SDA_GPIO_21
- net SDA_GPIO_21: now also D5.1 (I/O_1)
- net TXD0 renamed TXD0_GPIO_1
- net TXD0_GPIO_1: now also D5.5 (I/O_4)
- new net: C9.1, R18.1, Y1.1
- new net: C8.1, R19.1, Y1.2
- new net Inductive Loop/555TIMER-OUT_1: TP6.1
- new net Inductive Loop/555TIMER-OUT_2: TP5.1
- new net Inductive Loop/555TIMER-OUT_3: TP4.1
- new net TMS_GPIO_14: J1.9 (Pin_9), U2.13 (IO14)
- no-connect marks 14 -> 16
Other:
- note added: "GPIO ESD Protection"
- note added: "RTC Clock Source (Optional)"
- moved on the sheet: C10, C11, C12, C13, C14, C4, C5, C6, C7, D1, D2, D3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

Commit message: nothing
Parts:
- removed TP2: DTR, TestPoint:TestPoint_Bridge_Pitch2.54mm_Drill0.7mm, symbol Connector:TestPoint_2Pole
- removed TP3: RTS, TestPoint:TestPoint_Bridge_Pitch2.54mm_Drill0.7mm, symbol Connector:TestPoint_2Pole
- removed TP4: LOOP_OUT_3, TestPoint:TestPoint_Bridge_Pitch2.54mm_Drill0.7mm, symbol Connector:TestPoint_2Pole
- removed TP5: LOOP_OUT_2, TestPoint:TestPoint_Bridge_Pitch2.54mm_Drill0.7mm, symbol Connector:TestPoint_2Pole
- removed TP6: LOOP_OUT_1, TestPoint:TestPoint_Bridge_Pitch2.54mm_Drill0.7mm, symbol Connector:TestPoint_2Pole
- added R20: 5 MΩ, Resistor_SMD:R_0402_1005Metric, symbol Device:R
- added TP2: DTR, TestPoint:TestPoint_Bridge_Pitch2.54mm_Drill0.7mm, symbol Connector:TestPoint
- added TP3: RTS, TestPoint:TestPoint_Bridge_Pitch2.54mm_Drill0.7mm, symbol Connector:TestPoint
- added TP4: LOOP_OUT_3, TestPoint:TestPoint_Bridge_Pitch2.54mm_Drill0.7mm, symbol Connector:TestPoint
- added TP5: LOOP_OUT_2, TestPoint:TestPoint_Bridge_Pitch2.54mm_Drill0.7mm, symbol Connector:TestPoint
- added TP6: LOOP_OUT_1, TestPoint:TestPoint_Bridge_Pitch2.54mm_Drill0.7mm, symbol Connector:TestPoint
- C2: footprint (none) -> Capacitor_SMD:C_0402_1005Metric
- C8, C9: value 12pF/50V -> 8.2pF; footprint (none) -> Capacitor_SMD:C_0402_1005Metric; LCSC Part (none) -> C2857971
- J1: footprint (none) -> Connector_PinSocket_2.54mm:PinSocket_1x10_P2.54mm_Horizontal
- J2, J3: footprint (none) -> Connector_PinSocket_2.54mm:PinSocket_1x04_P2.54mm_Horizontal
- J4: footprint (none) -> Connector_PinSocket_2.54mm:PinSocket_2x07_P2.54mm_Horizontal
- Y1: value 32.768kHz -> 32.768kHz 7pF; footprint (none) -> Crystal:Crystal_SMD_2012-2Pin_2.0x1.2mm_HandSoldering; LCSC Part (none) -> C2905364
- renumbered R20 to R21, R21 to R22, R22 to R23, R23 to R24, R24 to R25, R25 to R26, R26 to R27, R27 to R28, R28 to R29, R29 to R30, R30 to R31, R31 to R32
Connections:
- net LOOP_OUT_1: now also TP6.1
- net LOOP_OUT_2: now also TP5.1
- net LOOP_OUT_3: now also TP4.1
- net at Q2.1 (E), R28.1, U3.4 (~{DTR}): now also TP2.1
- net at Q1.1 (E), R29.1, U3.6 (~{RTS}): now also TP3.1
- net at C9.1, R18.1, Y1.1: now also R20.2
- net at C8.1, R19.1, Y1.2: now also R20.1
- no-connect marks 16 -> 18
Other:
- sheet Power Interface ports: added I2C_SCL, I2C_SDA; removed USB D+, USB D-
- moved on the sheet: C8, C9, Y1
