File: kicad/Power_Interface.kicad_sch (KiCad schematic)
At the start: 26 parts, among them J8 USB-C Receptacle, U12 MAX40200AUK, U13 MX5052SL, U14 MX5052SL, U4 TLV76133DCY

Commit message: more updates
Parts:
- removed D7: TT0314TPX, easyeda2kicad:DFN2510-10_L2.5-W1.0-P0.50-BL, symbol EASYEDA2KICAD:TT0314TPX
- removed U13, U14: MX5052SL, easyeda2kicad:SOP-8_L5.1-W3.9-P1.27-LS6.0-BL, symbol EASYEDA2KICAD:MX5052SL
- added TP7: VBUSunreg, TestPoint:TestPoint_Bridge_Pitch2.54mm_Drill0.7mm, symbol Connector:TestPoint_2Pole
- added TP8: GND, TestPoint:TestPoint_Bridge_Pitch2.54mm_Drill0.7mm, symbol Connector:TestPoint_2Pole
- added TP9: 3V3, TestPoint:TestPoint_Bridge_Pitch2.54mm_Drill0.7mm, symbol Connector:TestPoint_2Pole
- renumbered C12 to C15, C9 to C16, C10 to C17, C11 to C18, C40 to C19, C38 to C20, C39 to C21, C2 to C22, D4 to D7, D6 to D8, R25 to R32, R43 to R33, R44 to R34, TP14 to TP10, U12 to U5
Connections:
- net +3.3V: now also TP9.2; no longer F1.1
- net GND: now also TP8.1; no longer C15.2, C19.2, U4.1 (GND)
- net VBUS_{unregulated}: now also TP7.2; no longer C15.1, U4.3 (VI)
- new net: F1.1, TP9.1
- new net: C15.1, TP7.1, U4.3 (VI)
- new net: C15.2, C19.2, TP8.2, U4.1 (GND)
Other:
- note removed: "GPIO_0 protected with 100Ω and 30mA polyfuse"
- note removed: "Ideal Diode Vf - 40mV"
- note removed: "TVS Diode 3.5V Clamping 3.3V Vrwm"
- moved on the sheet: C16, C17, C18, D7, F1, R32

Commit message: nothing
Parts:
- removed TP7: VBUSunreg, TestPoint:TestPoint_Bridge_Pitch2.54mm_Drill0.7mm, symbol Connector:TestPoint_2Pole
- removed TP8: GND, TestPoint:TestPoint_Bridge_Pitch2.54mm_Drill0.7mm, symbol Connector:TestPoint_2Pole
- removed TP9: 3V3, TestPoint:TestPoint_Bridge_Pitch2.54mm_Drill0.7mm, symbol Connector:TestPoint_2Pole
- added C20, C21: 100nF, Capacitor_SMD:C_0402_1005Metric, symbol Device:C_Small
- added R33: 0.05 1%, Resistor_SMD:R_2512_6332Metric, symbol Device:R
- added R34, R35: 10, Resistor_SMD:R_0402_1005Metric, symbol Device:R_Small
- added R36: 10k, Resistor_SMD:R_0402_1005Metric, symbol Device:R_Small
- added TP7: VBUSunreg, TestPoint:TestPoint_Bridge_Pitch2.54mm_Drill0.7mm, symbol Connector:TestPoint
- added TP8: LOOP_OUT_2, TestPoint:TestPoint_Bridge_Pitch2.54mm_Drill0.7mm, symbol Connector:TestPoint
- added TP9: 3V3, TestPoint:TestPoint_Bridge_Pitch2.54mm_Drill0.7mm, symbol Connector:TestPoint
- added U5: INA226, Package_SO:TSSOP-10_3x3mm_P0.5mm, symbol Sensor_Energy:INA226
- F1: footprint (none) -> Fuse:Fuse_1812_4532Metric; LCSC Part (none) -> C49318440
- renumbered C20 to C22, C21 to C23, C22 to C24, R32 to R37, R33 to R38, R34 to R39, U5 to U6
Connections:
- net +3.3V: now also C21.1, R33.1, R34.1, R36.2, TP9.1, U5.6 (VS)
- net GND: now also C15.2, C19.2, U4.1 (GND), C21.2, TP8.1, U5.1 (A1), U5.2 (A0), U5.7 (GND)
- net VBUS_{unregulated}: now also C15.1, U4.3 (VI), TP7.1
- net at F1.1: now also R33.2, R35.1, U5.8 (Vbus)
- new net: C20.2, R35.2, U5.10 (Vin+)
- new net: R36.1, U5.3 (~{Alert})
- new net: C20.1, R34.2, U5.9 (Vin-)
- new net I2C_SCL: U5.5 (SCL)
- new net I2C_SDA: U5.4 (SDA)
Other:
- moved on the sheet: D7, F1, H1, H2, H3, H4, R37
